File: hamtonio.sch (EAGLE design)
At the start: 52 parts, among them SW2 SPST_TACT-KMR2, U1 TPS61029_DRC_10, U4 AP2112-3.3, U5 TXB0104PWR, X5 32.768

Commit message: tft carrier and hamtonio mkx2; Oshpark MKiCLdFX
Parts:
- removed C17, C18: 0.1uF, microbuilder:CAP_CERAMIC0805-NOOUTLINE
- removed G2: 12BH311P-GR, POV_light:AA
- removed J2: (no value), SparkFun-Connectors:CONN_021X02_NO_SILK
- removed J5: (no value), SparkFun-Connectors:CONN_06NO_SILK_FEMALE_PTH
- removed LED2: (no value), adafruit:LEDCHIPLED-0603-TTW
- removed LED3: AP102-2020, microbuilder:APA1022020
- removed LO_BAT1: RD, SparkFun-LED:LED0603
- removed R11: 2.2K, microbuilder:RESISTOR_0603_NOOUT
- removed R14: 1.5M, resistor:R-US_R0805
- removed R15: 1M, resistor:R-US_R0805
- removed R16: 300, resistor:R-US_R0805
- removed R17: 165k, adafruit:R-US_R0805
- removed R18, R19: 390k, resistor:R-US_R0805
- removed SW2: SPST_TACT-KMR2, adafruit:SPST_TACT-KMR2
- removed U$14, U$16, U$19, U$5: FLAT_SMD_WIRE_PAD, 00_bsiepert:FLAT_SMD_WIRE_PAD
- removed U$20: WINDBOND_QSPI_FLASHWSON_6X5, 00_bsiepert:WINDBOND_QSPI_FLASHWSON_6X5
- removed U5: TXB0104PWR, microbuilder:TXB0104PWR
- added BT1: (no value), 00_bsiepert:BATTERYDUAL_AA_XX
- added C1: 0.1uF, SparkFun-Capacitors:0.1UF-0603-25V-(+80/-20%)
- added J6, J7: (no value), SparkFun-Connectors:CONN_08NO_SILK_FEMALE_PTH
- added QSPI: WINDBOND_QSPI_FLASHWSON_6X5, 00_bsiepert:WINDBOND_QSPI_FLASHWSON_6X5
- added R2: 330, adafruit:R-US_R0603
- added R3: 1k, adafruit:R-US_R0603
- added R5: 10k, adafruit:R-US_R0603
- added R7: 165k, adafruit:R-US_R0603
- added R8: 1.5M, adafruit:R-US_R0603
- added U$2: SWD_HEADER, 00_bsiepert:SWD_HEADER
- added U$22, U$34, U$39: MOUNTINGHOLE2.5, microbuilder:MOUNTINGHOLE2.5
- J1, J3, J4: device SparkFun-Connectors:CONN_021X02_NO_SILK -> SparkFun-Connectors:CONN_041X04_NO_SILK
- R1: value 10K -> 390k; device microbuilder:RESISTOR_0603_NOOUT -> adafruit:R-US_R0603
- R6: value 10K -> 390k; device microbuilder:RESISTOR0805_NOOUTLINE -> adafruit:R-US_R0603
- R9: value 1K -> 1M; device microbuilder:RESISTOR_0603_NOOUT -> adafruit:R-US_R0603
- U$12: value 10118193-0001LF -> AMPHENOL_MICRO_USBAMPHENOL_MICRO_USB_BETTER; device 00_bsiepert:AMPHENOL_MICRO_USB -> 00_bsiepert:AMPHENOL_MICRO_USBAMPHENOL_MICRO_USB_BETTER
Connections:
- net 13 renamed N$3
- net N$14 renamed SW
- removed net 10: U$1.PA21/XINT5/Y15/SERCOM5.3&3.3/I2S-SDO
- removed net 11: U$1.PA22/XINT6/Y16/SERCOM3.0&5.1/I2S-SDI
- removed net 12: U$1.PA23/XINT7/Y17/SRCOM3.1&5.0/USBSOF/CAN0RX/I2S-FS1
- removed net 4: U$1.PA27/XINTY18
- removed net 5: U$1.PA18/EXINT2/Y12/SERCOM1.2&3.2, U5.A2
- removed net 5!: J2.2, U5.B2
- removed net 7: U$1.PA19/EXINT3/Y13/SERCOM1.3&3.3, U5.A1
- removed net 7!: J2.1, U5.B1
- removed net 9: U$1.PA20/XINT4/Y14/SERCOM5.2&3.2/I2S-FS0
- removed net A0: J5.1, U$1.PA02/EINT2/AIN0/VOUT0
- removed net A1: J5.2, U$1.PB08/EXINT8/ADC0.2&1.0/Y1/SERCOM4.0
- removed net A2: J5.3, U$1.PB09/EXINT9/ADC0.3&1.1/Y2/SERCOM4.1
- removed net A3: J5.4, U$1.PA04/EINT4/VREFB/AIN4/Y3/SERCOM0.0
- removed net A4: J5.5, U$1.PA05/EINT5/AIN5/VOUT1/SERCOM0.1
- removed net D8: LO_BAT1.C, R16.1
- removed net DOT_MOSI: LED3.DI, U$1.PB02/XINT2/ADC0.14/Y20/SERCOM5.0
- removed net DOT_SCK: LED3.CKI, U$1.PB03/XINT3/ADC0.15/Y23/SRCOM5.1
- removed net MOSI: U$1.PA12/XINT12/SERCOM2.0&4.1
- removed net N$10: R18.1, R19.2, U1.LBI
- removed net N$13: R15.1, R16.2, U1.LBO
- removed net N$17: R14.1, R17.2, U1.FB
- removed net N$3 (its old number): U$1.PA07/EINT7/AIN7/Y5/SERCOM0.3
- removed net N$8: U$1.PA15/EXINT15/SERCOM2.3&4.3
- removed net N$9: LED2.A, R11.2
- removed net OE2: R6.1, U5.OE
- removed net SCK: U$1.PA13/XINT13/SERCOM2.1&4.0
- removed net SCL: U$1.PA17/EXINT1/Y11/SERCOM1.1&3.0, U5.A3
- removed net SCL!: J1.1, U5.B3
- removed net SDA: U$1.PA16/EXINT0/Y10/SERCOM1.0&3.1, U5.A4
- removed net SDA!: J1.2, U5.B4
- removed net SWCLK: R9.1, U$1.PA30/XINT14/Y19/SRCOM7.2+1.2/SWCLK, U$19.P$1
- removed net TX: U$1.PA06/EINT6/AIN6/Y4/SERCOM0.2
- removed net V+: C3.1, G2.+, L3.1, R18.2, U1.EN, U1.VBAT
- new net !RESET_SW: R2.2, U$2.RESET
- new net BOOST_EN: S1.P, U1.EN
- new net DAC_0: J3.1, U$1.PA02/EINT2/AIN0/VOUT0
- new net DAC_1: J3.2, J6.6, U$1.PA05/EINT5/AIN5/VOUT1/SERCOM0.1
- new net DOT_0_MOS: J1.2, U$1.PA13/XINT13/SERCOM2.1&4.0
- new net DOT_0_SCK: J1.1, U$1.PA12/XINT12/SERCOM2.0&4.1
- new net DOT_1_MOS: J4.2, U$1.PA17/EXINT1/Y11/SERCOM1.1&3.0
- new net DOT_1_SCK: J4.1, U$1.PA16/EXINT0/Y10/SERCOM1.0&3.1
- new net DOT_2_MOS: U$1.PB02/XINT2/ADC0.14/Y20/SERCOM5.0
- new net DOT_2_SCK: U$1.PB03/XINT3/ADC0.15/Y23/SRCOM5.1
- new net FB: R7.2, R8.1, U1.FB
- new net LBI: R1.2, R6.1, U1.LBI
- new net LBO: R9.1, U$1.PA15/EXINT15/SERCOM2.3&4.3, U1.LBO
- new net MISC_0: J7.1, U$1.PA18/EXINT2/Y12/SERCOM1.2&3.2
- new net MISC_1: J7.2, U$1.PA19/EXINT3/Y13/SERCOM1.3&3.3
- new net MISC_2: J7.3, U$1.PA20/XINT4/Y14/SERCOM5.2&3.2/I2S-FS0
- new net MISC_3: J7.4, U$1.PA21/XINT5/Y15/SERCOM5.3&3.3/I2S-SDO
- new net MISC_4: J7.5, U$1.PA22/XINT6/Y16/SERCOM3.0&5.1/I2S-SDI
- new net MISC_5: J7.6, U$1.PA23/XINT7/Y17/SRCOM3.1&5.0/USBSOF/CAN0RX/I2S-FS1
- new net SWDCLK: R3.2, U$1.PA30/XINT14/Y19/SRCOM7.2+1.2/SWCLK, U$2.SWDCLK
- new net TFT_CS: J6.3, U$1.PA04/EINT4/VREFB/AIN4/Y3/SERCOM0.0
- new net TFT_DC: J6.4, U$1.PA06/EINT6/AIN6/Y4/SERCOM0.2
- new net TFT_MOS: J6.2, U$1.PB08/EXINT8/ADC0.2&1.0/Y1/SERCOM4.0
- new net TFT_RST: J6.5, U$1.PA07/EINT7/AIN7/Y5/SERCOM0.3
- new net TFT_SCK: J6.1, U$1.PB09/EXINT9/ADC0.3&1.1/Y2/SERCOM4.1
- net !RESET: now also C1.1, R2.1, R5.1; no longer R1.1, SW2.P, SW2.P1
- net GND: now also BT1.-, C1.2, J1.3, J3.3, J4.3, J6.7, J7.7, QSPI.GND, R1.1, R7.1, S1.O, U$2.GND@1, U$2.GND@2, U$2.GND@3; no longer C17.2, C18.2, G2.-, J4.1, J4.2, LED2.C, LED3.GND, R17.1, R19.1, SW2.S, SW2.S1, U$16.P$1, U$20.GND, U5.GND
- net QSPI_CS: now also QSPI.CS; no longer U$20.CS
- net QSPI_IO0: now also QSPI.DI/IO0; no longer U$20.DI/IO0
- net QSPI_IO1: now also QSPI.DO/IO1; no longer U$20.DO/IO1
- net QSPI_IO2: now also QSPI.WP/IO2; no longer U$20.WP/IO2
- net QSPI_IO3: now also QSPI.HOLD/IO3; no longer U$20.HOLD/IO3
- net QSPI_SCK: now also QSPI.CLK; no longer U$20.CLK
- net SWDIO: now also U$2.SWDIO; no longer U$5.P$1
- net VBAT: now also BT1.+, C3.1, L3.1, R6.2, S1.S, U1.VBAT; no longer D2.A, S1.P
- net VDDIO: now also J1.4, J3.4, J4.4, J6.8, J7.8, QSPI.VCC, R3.1, R5.2, U$2.VCC; no longer C17.1, LED3.VDD, R1.2, R11.1, R6.2, R9.2, U$14.P$1, U$20.VCC, U5.VCCA
- net VIN: no longer C18.1, J3.1, J3.2, U5.VCCB
- net VOUT: now also D2.A, R8.2, R9.2; no longer LO_BAT1.A, R14.2, R15.2, S1.O
Other:
- moved on the sheet: C10, C11, C12, C13, C2, C3, C4, C5, C6, C7, C8, C9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

Commit message: backin' up
Parts:
- removed U1: TPS61029_DRC_10, TPS61026:TPS61026_DRC_10
- added U$8: TPS61029, 00_bsiepert:TPS61029
- R8: value 1.5M -> 1M
Connections:
- net BOOST_EN: now also U$8.EN; no longer U1.EN
- net FB: now also U$8.FB; no longer U1.FB
- net GND: now also U$8.GND, U$8.PAD, U$8.PGND, U$8.PS; no longer U1.GND, U1.PAD, U1.PGND, U1.PS
- net LBI: now also U$8.LBI; no longer U1.LBI
- net LBO: now also U$8.LBO; no longer U1.LBO
- net SW: now also U$8.SW; no longer U1.SW
- net VBAT: now also U$8.VBAT; no longer U1.VBAT
- net VOUT: now also U$8.VOUT; no longer U1.VOUT
Changed lines of the file:
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@@
 <?xml version="1.0" encoding="utf-8"?>
 <!DOCTYPE eagle SYSTEM "eagle.dtd">
-<eagle version="9.2.1">
+<eagle version="9.2.2">
 <drawing>
 <settings>
@@
 <part name="L1" library="00_bsiepert" deviceset="1007_INDUCTOR" device="" value="10uH"/>
 <part name="SJ1" library="00_bsiepert" deviceset="SOLDERJUMPER" device="CLOSED"/>
-<part name="U1" library="TPS61026" deviceset="TPS61026_DRC_10" device="" value="TPS61029_DRC_10"/>
 <part name="C3" library="resistor" deviceset="C-US" device="C0805K" value="10uF"/>
 <part name="C4" library="resistor" deviceset="C-US" device="C0805K" value="2.2 uF"/>
@@
 <part name="R6" library="adafruit" library_urn="urn:adsk.eagle:library:420" deviceset="R-US_" device="R0603" value="390k"/>
 <part name="R7" library="adafruit" library_urn="urn:adsk.eagle:library:420" deviceset="R-US_" device="R0603" value="165k"/>
-<part name="R8" library="adafruit" library_urn="urn:adsk.eagle:library:420" deviceset="R-US_" device="R0603" value="1.5M"/>
+<part name="R8" library="adafruit" library_urn="urn:adsk.eagle:library:420" deviceset="R-US_" device="R0603" value="1M"/>
 <part name="R9" library="adafruit" library_urn="urn:adsk.eagle:library:420" deviceset="R-US_" device="R0603" value="1M"/>
 <part name="J1" library="SparkFun-Connectors" library_urn="urn:adsk.eagle:library:513" deviceset="CONN_04" device="1X04_NO_SILK" package3d_urn="urn:adsk.eagle:package:38094/1"/>
@@
 <part name="J4" library="SparkFun-Connectors" library_urn="urn:adsk.eagle:library:513" deviceset="CONN_04" device="1X04_NO_SILK" package3d_urn="urn:adsk.eagle:package:38094/1"/>
 <part name="U$5" library="microbuilder" deviceset="GND" device=""/>
+<part name="U$8" library="00_bsiepert" deviceset="TPS61029" device=""/>
 </parts>
 <sheets>
@@
 <attribute name="VALUE" x="16.51" y="111.76" size="1.778" layer="96" rot="R270"/>
 </instance>
-<instance part="U1" gate="A" x="58.42" y="236.22" smashed="yes">
-<attribute name="NAME" x="40.9956" y="250.4186" size="2.0828" layer="95" ratio="6" rot="SR0"/>
-<attribute name="VALUE" x="40.0558" y="247.8786" size="2.0828" layer="96" ratio="6" rot="SR0"/>
-</instance>
 <instance part="C3" gate="G$1" x="20.32" y="233.68" smashed="yes">
 <attribute name="NAME" x="21.336" y="234.315" size="1.778" layer="95"/>
@@
 <attribute name="VALUE" x="120.396" y="142.24" size="1.27" layer="96"/>
 </instance>
+<instance part="U$8" gate="A" x="58.42" y="241.3" smashed="yes"/>
 </instances>
 <busses>
@@
 </segment>
 <segment>
-<pinref part="U1" gate="A" pin="PAD"/>
-<pinref part="U1" gate="A" pin="GND"/>
 <wire x1="60.96" y1="220.98" x2="63.5" y2="220.98" width="0.1524" layer="91"/>
-<pinref part="U1" gate="A" pin="PS"/>
-<pinref part="U1" gate="A" pin="PGND"/>
+<pinref part="GND14" gate="1" pin="GND"/>
 <wire x1="55.88" y1="220.98" x2="58.42" y2="220.98" width="0.1524" layer="91"/>
-<pinref part="GND14" gate="1" pin="GND"/>
 <wire x1="58.42" y1="220.98" x2="60.96" y2="220.98" width="0.1524" layer="91"/>
 <wire x1="60.96" y1="220.98" x2="60.96" y2="215.9" width="0.1524" layer="91"/>
+<junction x="60.96" y="220.98"/>
+<pinref part="U$8" gate="A" pin="PS"/>
+<pinref part="U$8" gate="A" pin="PGND"/>
 <junction x="58.42" y="220.98"/>
-<junction x="60.96" y="220.98"/>
+<pinref part="U$8" gate="A" pin="GND"/>
+<pinref part="U$8" gate="A" pin="PAD"/>
 </segment>
 <segment>
@@
 <wire x1="20.32" y1="251.46" x2="20.32" y2="243.84" width="0.1524" layer="91"/>
 <junction x="20.32" y="238.76"/>
-<pinref part="U1" gate="A" pin="VBAT"/>
 <wire x1="20.32" y1="243.84" x2="20.32" y2="238.76" width="0.1524" layer="91"/>
 <pinref part="L3" gate="G$1" pin="1"/>
@@
 <pinref part="S1" gate="1" pin="S"/>
 <wire x1="20.32" y1="251.46" x2="76.2" y2="251.46" width="0.1524" layer="91"/>
+<pinref part="U$8" gate="A" pin="VBAT"/>
 </segment>
 </net>
@@
 <net name="LBI" class="0">
 <segment>
-<pinref part="U1" gate="A" pin="LBI"/>
 <wire x1="45.72" y1="233.68" x2="45.72" y2="226.06" width="0.1524" layer="91"/>
 <wire x1="45.72" y1="226.06" x2="38.1" y2="226.06" width="0.1524" layer="91"/>
@@
 <junction x="38.1" y="226.06"/>
 <label x="45.72" y="228.6" size="1.778" layer="95" rot="R90"/>
+<pinref part="U$8" gate="A" pin="LBI"/>
 </segment>
 </net>
@@
 <wire x1="119.38" y1="208.28" x2="76.2" y2="208.28" width="0.1524" layer="91"/>
 <wire x1="76.2" y1="208.28" x2="76.2" y2="233.68" width="0.1524" layer="91"/>
-<pinref part="U1" gate="A" pin="LBO"/>
 <wire x1="76.2" y1="233.68" x2="73.66" y2="233.68" width="0.1524" layer="91"/>
 <junction x="119.38" y="208.28"/>
@@
 <label x="124.46" y="208.28" size="2.1844" layer="95"/>
 <pinref part="R9" gate="G$1" pin="1"/>
+<pinref part="U$8" gate="A" pin="LBO"/>
 </segment>
 <segment>
@@
 <segment>
 <pinref part="L3" gate="G$1" pin="2"/>
-<pinref part="U1" gate="A" pin="SW"/>
 <wire x1="40.64" y1="243.84" x2="45.72" y2="243.84" width="0.1524" layer="91"/>
 <label x="40.64" y="243.84" size="1.778" layer="95"/>
+<pinref part="U$8" gate="A" pin="SW"/>
+<wire x1="45.72" y1="241.3" x2="45.72" y2="243.84" width="0.1524" layer="91"/>
 </segment>
 </net>
 <net name="FB" class="0">
 <segment>
-<pinref part="U1" gate="A" pin="FB"/>
 <wire x1="73.66" y1="236.22" x2="78.74" y2="236.22" width="0.1524" layer="91"/>
 <wire x1="78.74" y1="236.22" x2="78.74" y2="228.6" width="0.1524" layer="91"/>
@@
 <pinref part="R8" gate="G$1" pin="1"/>
 <junction x="83.82" y="228.6"/>
+<pinref part="U$8" gate="A" pin="FB"/>
 </segment>
 </net>
 <net name="VOUT" class="0">
+<segment>
+<pinref part="D2" gate="G$1" pin="A"/>
+<wire x1="177.8" y1="241.3" x2="177.8" y2="248.92" width="0.1524" layer="91"/>
+<label x="177.8" y="241.3" size="1.27" layer="95" rot="R90"/>
+</segment>
 <segment>
 <pinref part="C5" gate="G$1" pin="+"/>
@@
 <wire x1="93.98" y1="238.76" x2="106.68" y2="238.76" width="0.1524" layer="91"/>
 <junction x="93.98" y="238.76"/>
-<pinref part="U1" gate="A" pin="VOUT"/>
 <wire x1="73.66" y1="238.76" x2="83.82" y2="238.76" width="0.1524" layer="91"/>
 <wire x1="83.82" y1="238.76" x2="93.98" y2="238.76" width="0.1524" layer="91"/>
@@
 <junction x="83.82" y="238.76"/>
 <pinref part="R9" gate="G$1" pin="2"/>
-</segment>
-<segment>
-<pinref part="D2" gate="G$1" pin="A"/>
-<wire x1="177.8" y1="241.3" x2="177.8" y2="248.92" width="0.1524" layer="91"/>
-<label x="177.8" y="241.3" size="1.27" layer="95" rot="R90"/>
+<pinref part="U$8" gate="A" pin="VOUT"/>
 </segment>
 </net>
@@
 <net name="BOOST_EN" class="0">
 <segment>
-<pinref part="U1" gate="A" pin="EN"/>
 <pinref part="S1" gate="1" pin="P"/>
 <wire x1="73.66" y1="243.84" x2="73.66" y2="241.3" width="0.1524" layer="91"/>
 <label x="73.66" y="241.3" size="1.778" layer="95"/>
-</segment>
-</net>
+<pinref part="U$8" gate="A" pin="EN"/>
+</segment>
+</net>
